File: EE/PCB UI ESP32/Display.kicad_sch (KiCad schematic)
At the start: 7 parts, among them U10 PESD3V3L1BA, U7 PESD3V3L1BA, U8 DW-20-07-T-S-200, U9 PESD3V3L1BA

Commit message: Finished first draft of ESP32-UI board
And moved around footprints, 3D models, etc. to match.
Parts:
- U10, U7, U9: footprint PESD3V3L1BA:SOD2512X110N -> DaisyBio_Mira:SOD2512X110N
- U8: footprint DW-20-07-T-S-200:HDRV20W64P0X254_1X20_5080X254X1067P -> DaisyBio_Mira:HDRV20W64P0X254_1X20_5080X254X1067P
Changed lines of the file:
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@@
 			)
 		)
-		(property "Footprint" "PESD3V3L1BA:SOD2512X110N"
+		(property "Footprint" "DaisyBio_Mira:SOD2512X110N"
 			(at 73.66 132.715 0)
 			(effects
@@
 			)
 		)
-		(property "Footprint" "PESD3V3L1BA:SOD2512X110N"
+		(property "Footprint" "DaisyBio_Mira:SOD2512X110N"
 			(at 109.855 132.08 0)
 			(effects
@@
 			)
 		)
-		(property "Footprint" "DW-20-07-T-S-200:HDRV20W64P0X254_1X20_5080X254X1067P"
+		(property "Footprint" "DaisyBio_Mira:HDRV20W64P0X254_1X20_5080X254X1067P"
 			(at 66.675 50.165 0)
 			(effects
@@
 			)
 		)
-		(property "Footprint" "PESD3V3L1BA:SOD2512X110N"
+		(property "Footprint" "DaisyBio_Mira:SOD2512X110N"
 			(at 48.26 132.715 0)
 			(effects

Commit message: Finished V1 of ESP-UI
This is the version of ESP-UI that was ordered July 20 2025.
Parts:
- U8: Value_1 DW-20-07-T-S-200 -> NHD-0420CW-AW3
Changed lines of the file:
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@@
 			)
 		)
-		(property "Value_1" "DW-20-07-T-S-200"
+		(property "Value_1" "NHD-0420CW-AW3"
 			(at 90.805 31.75 90)
 			(effects
